Commit message: CambiosGenerales_29/07/2023

File: description/robot.urdf.xacro (robot description, xacro)
@@ -1,7 +1,7 @@
 <?xml version="1.0"?>
-<robot xmlns:xacro="http://www.ros.org/wiki/xacro"  name="robot">
+<robot xmlns:xacro="http://www.ros.org/wiki/xacro" name="robot">
     <!-- Example link -->
+    <xacro:include filename="properties.xacro"/>
     <xacro:include filename="robot_core.xacro"/>
-        <!-- Example link -->
-    <link name="base_link"></link>
+    <xacro:include filename="inertial_macros.xacro"/>
 </robot>

Commit message: cambios faltantes 4 de agosto 2023

File: description/robot.urdf.xacro (robot description, xacro)
@@ -5,3 +5,4 @@
     <xacro:include filename="robot_core.xacro"/>
     <xacro:include filename="inertial_macros.xacro"/>
+    <xacro:include filename="gazebo_control.xacro"/>
 </robot>

File: description/robot_core.xacro (robot description, xacro)
@@ -29,4 +29,7 @@
             <origin xyz="0.15 0 0.075" rpy="0 0 0"/>
         </xacro:inertial_box>
+        <gazebo reference="chassis">
+            <material>Gazebo/White</material>
+        </gazebo>
     </link>
     <!-- left wheel joint -->
@@ -53,4 +56,7 @@
             <origin xyz="0 0 0" rpy="0 0 0"/>
         </xacro:inertial_cylinder>
+        <gazebo reference="left_wheel">
+            <material>Gazebo/Blue</material>
+        </gazebo>
     </link>
     <!-- right wheel joint -->
@@ -77,4 +83,7 @@
             <origin xyz="0 0 0" rpy="0 0 0"/>
         </xacro:inertial_cylinder>
+        <gazebo reference="right_wheel">
+            <material>Gazebo/Blue</material>
+        </gazebo>
     </link>
     <!-- caster wheel joint -->
@@ -100,4 +109,9 @@
             <origin xyz="0 0 0" rpy="0 0 0"/>
         </xacro:inertial_sphere>
+        <gazebo reference="caster_wheel">
+            <material>Gazebo/Black</material>
+            <mu1 value = "0.001" />
+            <mu2 value = "0.001" />
+        </gazebo>
     </link>
 </robot>
