Commit message: en clase 5 agosto 2023

File: description/robot_core.xacro (robot description, xacro)
@@ -29,8 +29,8 @@
             <origin xyz="0.15 0 0.075" rpy="0 0 0"/>
         </xacro:inertial_box>
-        <gazebo reference="chassis">
+    </link>
+    <gazebo reference="chassis">
             <material>Gazebo/White</material>
         </gazebo>
-    </link>
     <!-- left wheel joint -->
     <joint name="left_wheel_joint" type="continuous">
@@ -56,8 +56,8 @@
             <origin xyz="0 0 0" rpy="0 0 0"/>
         </xacro:inertial_cylinder>
-        <gazebo reference="left_wheel">
+    </link>
+    <gazebo reference="left_wheel">
             <material>Gazebo/Blue</material>
         </gazebo>
-    </link>
     <!-- right wheel joint -->
     <joint name="right_wheel_joint" type="continuous">
@@ -83,8 +83,8 @@
             <origin xyz="0 0 0" rpy="0 0 0"/>
         </xacro:inertial_cylinder>
-        <gazebo reference="right_wheel">
-            <material>Gazebo/Blue</material>
+    </link>
+    <gazebo reference="right_wheel">
+        <material>Gazebo/Blue</material>
         </gazebo>
-    </link>
     <!-- caster wheel joint -->
     <joint name="caster_wheel_joint" type="fixed">
@@ -109,4 +109,5 @@
             <origin xyz="0 0 0" rpy="0 0 0"/>
         </xacro:inertial_sphere>
+    </link>
         <gazebo reference="caster_wheel">
             <material>Gazebo/Black</material>
@@ -114,4 +115,3 @@
             <mu2 value = "0.001" />
         </gazebo>
-    </link>
 </robot>
