Commit message: ultima clase

File: description/lidar.xacro (robot description, xacro)
@@ -47,5 +47,5 @@
             <plugin name="laser_controller" filename="libgazebo_ros_ray_sensor.so">
                 <ros>
-                    <argument>--ros-args --remap ~/out:=scan</argument>
+                    <argument>~/out:=scan</argument>
                 </ros>
                 <output_type>sensor_msgs/LaserScan</output_type>

File: description/robot_core.xacro (robot description, xacro)
@@ -11,4 +11,12 @@
         <origin xyz="-0.1 0 0"/>
     </joint>
+    <!-- base_footprint joint -->
+    <joint name="base_footprint_joint" type="fixed">
+        <parent link="base_link"/>
+        <child link="base_footprint"/>
+        <origin xyz="0 0 -0.025"/>
+    </joint>
+    <link name="base_footprint">
+    </link>
     <!-- chassis link -->
     <link name="chassis">
